File: AmplificadorDeInstrumentacion.kicad_sch (KiCad schematic)
At the start: 23 parts, among them Q1 TIP31, Q2 TIP32, U1 LF357, U2 LF357, U3 OPAMP, U4 OPAMP, U5 OPAMP

Commit message: feat: update simulation results and project files for instrumentation amplifier characterization
Parts:
- U1, U2: value LF357 -> OPAMP
Connections:
- net +15V: now also RL.2, Rb1.2; no longer RL.1, Rb1.1
- net -15V: now also Rb2.1; no longer Rb2.2
- net GND: now also R6.1, R9.1; no longer Cf.2, R6.2, R9.2
- net at D2.2 (A), Q2.B: now also Rb2.2; no longer Rb2.1
- net at R5.2, U3.2 (-): now also R6.2; no longer R6.1
- net at D1.1 (K), Q1.B: now also Rb1.1; no longer Rb1.2
- net at R10.1, U4.3 (+): now also R9.2; no longer R9.1
- net at Rf.2, U5.2 (-): no longer Cf.1
- net at R2.1, U2.3 (+): now also Rg.1; no longer Rg.2
- net at R1.1, U1.3 (+): now also Rg.2; no longer Rg.1
